File: custom_pcb/bikesensor_pcb/bikesensor_pcb.kicad_sch (KiCad schematic)
At the start: 18 parts, among them J1 ESP32_Left, J2 ESP32_Right, J3 MPU6050, J4 SD_Breakout, J5 NEO-6M_GPS, J6 Conn_01x08_Socket, J7 Conn_01x08_Socket, J8 Conn_01x01, SW1 SW1

Commit message: Shrink the carrier board to the real module footprints
Re-lays the board out against the actual ESP32-C3 SuperMini and Wemos
battery shield dimensions: ESP32 rows J1-J2 go 800 -> 600 mil, shield
rows J6-J7 go 1000 -> 900 mil, and the outline drops from 72.75 x 167.43
to 38.74 x 114.47 mm -- the size the README already claimed. Mounting
holes H1-H4 are dropped along with the reclaimed area.

KiCad is not installed on this machine, so this was verified by
rebuilding the connectivity graph straight from the file: every pad sits
at least 1.16 mm inside the board edge, and every net is fully routed
except +3V3, whose track stops 1.48 mm short of C1 pin 1. That bulk cap
is still floating and needs one more track before this is fabbed.

Co-Authored-By: Claude Opus 5 <noreply@anthropic.com>
Claude-Session: https://claude.ai/code/session_01EcNmG8boCU9EBpJGftDikR
Parts:
- removed H1, H2, H3, H4: MountingHole, MountingHole:MountingHole_5.3mm_M5, symbol Mechanical:MountingHole

Commit message: Add the CS pull-up and close the two open nets
R3 (10k, /SPI_CS to +3V3) is in the design, and +3V3 now reaches C1
pin 1. Verified from the file rather than from DRC's word for it:
0 unrouted nets across the whole board, and R3's pads land on +3V3
and /SPI_CS.

Also re-aligns the J4 MOSI and SCK silkscreen labels. They had drifted
3.46 mm and 2.92 mm down while the silk overlaps were being cleared,
which put MOSI beside the SCK pin and SCK beside the CS pin -- wiring
the SD card from those labels would have swapped the SPI lines. All six
J4 labels now sit exactly on their pads.

Co-Authored-By: Claude Opus 5 <noreply@anthropic.com>
Claude-Session: https://claude.ai/code/session_01EcNmG8boCU9EBpJGftDikR
Parts:
- added R3: 10k, Resistor_THT:R_Axial_DIN0207_L6.3mm_D2.5mm_P7.62mm_Horizontal, symbol Device:R
Connections:
- net +3V3: now also R3.2
- net SPI_CS: now also R3.1
Changed lines of the file:
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@@
 	(wire
 		(pts
+			(xy 173.99 45.72) (xy 173.99 50.8)
+		)
+		(stroke
+			(width 0)
+			(type default)
+		)
+	)
+	(wire
+		(pts
 			(xy 99.06 63.5) (xy 110.49 63.5)
 		)
@@
 	(wire
 		(pts
+			(xy 166.37 58.42) (xy 173.99 58.42)
+		)
+		(stroke
+			(width 0)
+			(type default)
+		)
+	)
+	(wire
+		(pts
 			(xy 97.79 81.28) (xy 110.49 81.28)
 		)
@@
 		)
 	)
+	(label "SPI_CS"
+		(at 173.99 45.72 0)
+		(effects
+			(font
+				(size 1.27 1.27)
+			)
+			(justify left bottom)
+		)
+	)
 	(label "UART_TX_DEBUG"
 		(at 97.79 106.68 0)
@@
 	)
 	(symbol
+		(lib_id "power:+3V3")
+		(at 166.37 58.42 0)
+		(unit 1)
+		(body_style 1)
+		(exclude_from_sim no)
+		(in_bom yes)
+		(on_board yes)
+		(in_pos_files yes)
+		(dnp no)
+		(fields_autoplaced yes)
+		(property "Reference" "#PWR018"
+			(at 166.37 62.23 0)
+			(hide yes)
+			(show_name no)
+			(do_not_autoplace no)
+			(effects
+				(font
+					(size 1.27 1.27)
+				)
+			)
+		)
+		(property "Value" "+3V3"
+			(at 166.37 53.34 0)
+			(show_name no)
+			(do_not_autoplace no)
+			(effects
+				(font
+					(size 1.27 1.27)
+				)
+			)
+		)
+		(property "Footprint" ""
+			(at 166.37 58.42 0)
+			(hide yes)
+			(show_name no)
+			(do_not_autoplace no)
+			(effects
+				(font
+					(size 1.27 1.27)
+				)
+			)
+		)
+		(property "Datasheet" ""
+			(at 166.37 58.42 0)
+			(hide yes)
+			(show_name no)
+			(do_not_autoplace no)
+			(effects
+				(font
+					(size 1.27 1.27)
+				)
+			)
+		)
+		(property "Description" "Power symbol creates a global label with name \"+3V3\""
+			(at 166.37 58.42 0)
+			(hide yes)
+			(show_name no)
+			(do_not_autoplace no)
+			(effects
+				(font
+					(size 1.27 1.27)
+				)
+			)
+		)
+		(pin "1"
+		)
+		(instances
+			(project "bikesensor_pcb"
+				(path "/92844cda-fb34-4359-9dbb-e14c64aaab65"
+					(reference "#PWR018")
+					(unit 1)
+				)
+			)
+		)
+	)
+	(symbol
 		(lib_id "Device:C")
 		(at 160.02 146.05 0)
@@
 					(unit 1)
 				)
+			)
+		)
+	)
+	(symbol
+		(lib_id "Device:R")
+		(at 173.99 54.61 0)
+		(unit 1)
+		(body_style 1)
+		(exclude_from_sim no)
+		(in_bom yes)
+		(on_board yes)
+		(in_pos_files yes)
+		(dnp no)
+		(fields_autoplaced yes)
+		(property "Reference" "R3"
+			(at 176.53 53.3399 0)
+			(show_name no)
+			(do_not_autoplace no)
+			(effects
+				(font
+					(size 1.27 1.27)
+				)
+				(justify left)
+			)
+		)
+		(property "Value" "10k"
+			(at 176.53 55.8799 0)
+			(show_name no)
+			(do_not_autoplace no)
+			(effects
+				(font
+					(size 1.27 1.27)
+				)
+				(justify left)
+			)
+		)
+		(property "Footprint" "Resistor_THT:R_Axial_DIN0207_L6.3mm_D2.5mm_P7.62mm_Horizontal"
+			(at 172.212 54.61 90)
+			(hide yes)
+			(show_name no)
+			(do_not_autoplace no)
+			(effects
+				(font
+					(size 1.27 1.27)
+				)
+			)
+		)
+		(property "Datasheet" ""
+			(at 173.99 54.61 0)
+			(hide yes)
+			(show_name no)
+			(do_not_autoplace no)
+			(effects
+				(font
+					(size 1.27 1.27)
+				)
+			)
+		)
+		(property "Description" "Resistor"
+			(at 173.99 54.61 0)
+			(hide yes)
+			(show_name no)
+			(do_not_autoplace no)
+			(effects
+				(font
+					(size 1.27 1.27)
+				)
+			)
+		)
+		(pin "2"
+		)
+		(pin "1"
+		)
+		(instances
+			(project "bikesensor_pcb"
+				(path "/92844cda-fb34-4359-9dbb-e14c64aaab65"
+					(reference "R3")
+					(unit 1)
+				)
